File: Power Suply.kicad_pcb (KiCad board)
At the start: 2 copper layers, 120 x 75 mm, 23 parts, among them J1 Screw_Terminal_01x02, J2 Screw_Terminal_01x02, J3 Screw_Terminal_01x02, Q1 TIP41C, Q2 TIP41C

Commit message: Images
Parts:
- moved C4 5.00 mm to (215.7, 132.5)
- moved C5 5.00 mm to (175.8, 132.5)
- moved D5 5.00 mm to (190.4, 127.4)
- moved D6 5.00 mm to (215.7, 114.9)
- moved J3 5.00 mm to (162.0, 135.8)
- moved Q2 5.00 mm to (190.4, 114.9)
- moved R4 5.00 mm to (175.8, 122.5)
- moved J2 5.00 mm to (233.0, 127.7)
Routing:
- net Net-(Q1-C): track 252.0 -> 209.7 mm, vias 2 -> 0
- net Net-(D7-K): track 53.1 -> 48.1 mm
- net Net-(D10-A): track 51.1 -> 46.1 mm
- net GND: track 234.7 -> 229.7 mm
Other:
- board size 120 x 75 mm -> 120 x 70 mm
